File: NIVARA KICAD/Kicad/Nivara proyecto Electiva/NIVARA PROJECT/NIVARA PROJECT.kicad_pcb (KiCad board)
At the start: 2 copper layers, 102.2 x 83 mm, 100 parts, among them K1 G2RL-1, K2 G2RL-1, Q1 NCV8402xST, Q2 NCV8402xST, Q3 NCV8402xST, Q4 NCV8402xST, T1 IRF9310TRPBF, U1 GP8303-TC50-EW, U10 LTV-357TB, U11 LTV-357TB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

Commit message: Add files via upload
Parts:
- moved R2 206.4 mm to (193.6, 78.6)
- moved R1 204.6 mm to (182.3, 123.8), turned to -90 degrees
- moved R12 181.2 mm to (159.9, 107.5), turned to 180 degrees
- moved C11 178.0 mm to (155.9, 111.5), turned to 90 degrees
- moved R13 176.9 mm to (155.9, 107.5)
- moved C5 129.7 mm to (133.7, 125.3)
- moved C1 127.8 mm to (114.5, 96.6)
- moved L1 124.8 mm to (123.2, 124.8)
- moved R35 123.5 mm to (155.1, 70.9), turned to 180 degrees
- moved JP1 121.5 mm to (129.2, 124.5), turned to 90 degrees
- moved R36 121.0 mm to (155.0, 67.7), turned to 180 degrees
- moved C6 119.0 mm to (132.5, 114.0)
- moved R4 114.6 mm to (132.7, 120.8)
- moved R3 114.0 mm to (132.7, 117.3)
- moved U17 112.7 mm to (123.2, 117.3)
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Connections:
- D2 pad 1: VCC -> +3.3V
- K1 pad A1: VCC -> +3.3V
- K2 pad A1: VCC -> +3.3V
- Q1 pad 3: NPNOUT_GND -> GND
- Q2 pad 1: NPNOUT_GND -> GND
- Q2 pad 3: NPNOUT_GND -> GND
- Q3 pad 3: PNPOUT_GND -> GND
- Q4 pad 3: PNPOUT_GND -> GND
- R16 pad 1: NPNOUT_GND -> GND
- R17 pad 2: NPNOUT_GND -> GND
- R22 pad 2: VCC -> +3.3V
- R24 pad 2: VCC -> +3.3V
- R31 pad 2: PNPOUT_GND -> GND
- R33 pad 2: PNPOUT_GND -> GND
- U1 pad 5: VCC -> +3.3V
- U12 pad 2: PNPIN_GND -> GND
- U13 pad 2: PNPIN_GND -> GND
- U14 pad 4: PNP_VCC -> +3.3V
- U15 pad 4: PNP_VCC -> +3.3V
- U16 pad 5: VCC -> +3.3V
- U4 pad 4: VCC -> +3.3V
- U6 pad 3: NPNOUT_GND -> GND
- U6 pad 4: NPN_VCC -> +3.3V
- U7 pad 4: NPN_VCC -> +3.3V
- U8 pad 2: PNPIN_GND -> GND
- U9 pad 2: PNPIN_GND -> GND
Routing:
- net /BOARD_NIVARA/VOLTAGE_OUT/SDA: track 0.00 -> 144.2 mm, vias 0 -> 6
- net /BOARD_NIVARA/VOLTAGE_OUT/SCLK: track 0.00 -> 118.1 mm, vias 0 -> 6
- net /BOARD_NIVARA/A010_IN_1: track 0.00 -> 100.8 mm
- net /BOARD_NIVARA/NPN_OUT_1: track 0.00 -> 100.2 mm, vias 0 -> 2
- net /BOARD_NIVARA/relay/RL2_EN: track 0.00 -> 99.3 mm, vias 0 -> 6
- net /BOARD_NIVARA/A420_IN1: track 0.00 -> 93.8 mm, vias 0 -> 2
- net /BOARD_NIVARA/relay/RL1_EN: track 0.00 -> 88.7 mm, vias 0 -> 4
- net /BOARD_NIVARA/NPN_OUT_2: track 0.00 -> 82.6 mm, vias 0 -> 4
- net /BOARD_NIVARA/DRIVER-485/UART_OUT: track 0.00 -> 74.7 mm, vias 0 -> 4
- net /BOARD_NIVARA/DRIVER-485/UART_IN: track 0.00 -> 73.7 mm, vias 0 -> 6
- net GND: track 0.00 -> 59.3 mm, vias 0 -> 60
- net /BOARD_NIVARA/PNP_IN/NPN_OUT_D: track 0.00 -> 57.5 mm, vias 0 -> 4
- net /BOARD_NIVARA/NPN_IN/NPN_OUT_C: track 0.00 -> 54.8 mm, vias 0 -> 6
- net Net-(JP4-B): track 0.00 -> 54.2 mm
- net /BOARD_NIVARA/RS_485_A: track 0.00 -> 50.3 mm, vias 0 -> 6
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- added copper zone on In2.Cu, net +3.3V
- added copper zone on In1.Cu, net GND
- added copper zone on In2.Cu, net VCC
Other:
- copper layers 2 -> 4
- board text added: "10v in"
- board text added: "32v in"
- board text added: "Electiva para Meca"
- board text added: "Fausto Jimenez"
- board text added: "mA out"
- board text added: "npn in"
- board text added: "relay"
- board text added: "voltage out"
