File: NIVARA KICAD/Kicad/Nivara proyecto Electiva/NIVARA PROJECT/NIVARA PROJECT.kicad_sch (KiCad schematic)
At the start: 14 parts

Commit message: Add files via upload
Other:
- moved on the sheet: AE1
Changed lines of the file:
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@@
 	(symbol
 		(lib_id "Device:Antenna")
-		(at 194.31 52.07 0)
+		(at 195.58 52.07 0)
 		(unit 1)
 		(exclude_from_sim no)
@@
 		(fields_autoplaced yes)
 		(property "Reference" "AE1"
-			(at 196.85 51.4349 0)
+			(at 198.12 51.4349 0)
 			(effects
 				(font
@@
 		)
 		(property "Value" "WIFI-BT"
-			(at 196.85 53.9749 0)
+			(at 198.12 53.9749 0)
 			(effects
 				(font
@@
 		)
 		(property "Footprint" ""
-			(at 194.31 52.07 0)
+			(at 195.58 52.07 0)
 			(effects
 				(font
@@
 		)
 		(property "Datasheet" "~"
-			(at 194.31 52.07 0)
+			(at 195.58 52.07 0)
 			(effects
 				(font
@@
 		)
 		(property "Description" "Antenna"
-			(at 194.31 52.07 0)
+			(at 195.58 52.07 0)
 			(effects
 				(font
