File: NIVARA KICAD/Kicad/Nivara proyecto Electiva/NIVARA PROJECT/NPN_OUT.kicad_sch (KiCad schematic)
At the start: 8 parts, among them Q1 NCV8402xST, Q2 NCV8402xST, U6 LTV-357T, U7 LTV-357T

Commit message: Add files via upload
Connections:
- net NPNOUT_GND is gone; now on net GND: Q1.3 (S), Q2.1 (G), Q2.3 (S), R16.1, R17.2, U6.3
- net NPN_VCC renamed +3.3V
