File: NIVARA KICAD/Kicad/Nivara proyecto Electiva/NIVARA PROJECT/VOLTAGE_OUT.kicad_sch (KiCad schematic)
At the start: 5 parts, among them U4 GP8201S-TC50-EW

Commit message: Add files via upload
Connections:
- net VCC renamed +3.3V
Changed lines of the file:
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@@
 	)
 	(symbol
-		(lib_id "power:VCC")
+		(lib_id "power:+3.3V")
 		(at 123.19 83.82 90)
 		(unit 1)
@@
 			)
 		)
-		(property "Value" "VCC"
+		(property "Value" "+3.3V"
 			(at 119.38 83.8199 90)
 			(effects
@@
 			)
 		)
-		(property "Description" "Power symbol creates a global label with name \"VCC\""
+		(property "Description" "Power symbol creates a global label with name \"+3.3V\""
 			(at 123.19 83.82 0)
 			(effects
@@
 		)
 		(instances
-			(project ""
+			(project "NIVARA PROJECT"
 				(path "/dc6fb271-dfd0-4448-98f1-862b1cc93a80/2ca62569-d560-4cca-9470-52fd378086ae/4c56bdff-2384-434c-a91f-ac1414e948f2"
 					(reference "#PWR016")
