File: NIVARA KICAD/Kicad/Nivara proyecto Electiva/NIVARA PROJECT/mA_OUT.kicad_sch (KiCad schematic)
At the start: 18 parts, among them T1 IRF9310TRPBF, U1 GP8303-TC50-EW

Commit message: Add files via upload
Connections:
- net VCC renamed +3.3V
